Commit message: Fixed issues

File: gate_system/urdf/gate_system.urdf (robot description, URDF)
Before this commit: robot gate_system, 2 links, 1 joints
Links:
- added link world
- link base_link: mass 110.87 -> 1100.87
- link rotating_link: mass 1.2463 -> 0.1
Joints:
- added joint fixed: type fixed, parent world, child base_link, origin xyz=0 0 0 rpy=0 0 0

File: sjtu_drone/urdf/sjtu_drone.urdf (robot description, URDF)
Before this commit: robot sjtu_drone, 1 links, 0 joints
Links:
- link base_link: geometry collision mesh filename=package://sjtu_drone/models/sjtu_drone/quadrotor_4.stl; visual mesh filename=package://sjtu_drone/models/sjtu_drone/quadrotor_4.dae
